Commit message: modify second training

File: srs_training/urdf/box_world.urdf.xacro (robot description, xacro)
@@ -17,22 +17,11 @@
 	</link>
 	<link name="box1">
-		<inertial>
-		 <origin xyz="0 0 0.5" rpy="0 0 0"/>
-		 <mass value="1"/>
-		 <inertia ixx="100"  ixy="0"  ixz="0" iyy="100" iyz="0" izz="100" />
-		</inertial>
 		<visual>
 		 <origin xyz="0 0 0" rpy="0 0 0" />
 		 <geometry>
-		   <box size="1 1 1" />
+		   <box size="1 0.5 1" />
 		 </geometry>
 		 <material name="Red"/>
 		</visual>
-		<collision>
-		 <origin xyz="0 0 0" rpy="0 0 0"/>
-		 <geometry>
-		   <cylinder radius="1" length="0.5"/>
-		 </geometry>
-		</collision>
 	</link>
 	<joint name="box1_joint" type="fixed">

Commit message: Initial modifications to the robot urdf and callback for teleoperation

File: srs_training/urdf/box_world.urdf.xacro (robot description, xacro)
@@ -25,6 +25,6 @@
 		</visual>
 	</link>
-	<joint name="box1_joint" type="fixed">
-		<origin xyz="0 0 1" rpy="0 0 3.1416"/>
+	<joint name="box1_joint" type="planar">
+		<origin xyz="0 0 0.5" rpy="0 0 3.1416"/>
 		<parent link="base_link"/>
 		<child link="box1"/>

Commit message: 2nd SRS Training - Controlling movement inside gazebo and rviz

File: srs_training/urdf/box_world.urdf.xacro (robot description, xacro)
@@ -25,5 +25,5 @@
 		</visual>
 	</link>
-	<joint name="box1_joint" type="planar">
+	<joint name="box1_joint" type="floating">
 		<origin xyz="0 0 0.5" rpy="0 0 3.1416"/>
 		<parent link="base_link"/>

Commit message: training for navigation input

File: srs_training/urdf/box_world.urdf.xacro (robot description, xacro)
@@ -7,5 +7,5 @@
 	<!-- common stuff -->
 	<include filename="$(find cob_description)/urdf/materials.urdf.xacro" />
-	<link name="base_link">
+	<link name="map">
 		<visual>
 		 <origin xyz="0 0 0" rpy="0 0 0" />
@@ -16,17 +16,17 @@
 		</visual>
 	</link>
-	<link name="box1">
+	<link name="base_link">
 		<visual>
 		 <origin xyz="0 0 0" rpy="0 0 0" />
 		 <geometry>
-		   <box size="1 0.5 1" />
+		   <box size="1 0.5 0.5" />
 		 </geometry>
 		 <material name="Red"/>
 		</visual>
 	</link>
-	<joint name="box1_joint" type="floating">
+	<joint name="base_joint" type="floating">
 		<origin xyz="0 0 0.5" rpy="0 0 3.1416"/>
-		<parent link="base_link"/>
-		<child link="box1"/>
+		<parent link="map"/>
+		<child link="base_link"/>
 	</joint>
 </robot>

Commit message: training with robot mesh

File: srs_training/urdf/box_world.urdf.xacro (robot description, xacro)
@@ -9,22 +9,23 @@
 	<link name="map">
 		<visual>
-		 <origin xyz="0 0 0" rpy="0 0 0" />
-		 <geometry>
-		   <box size="10 10 0.1" />
-		 </geometry>
-		 <material name="Blue"/>
+			<origin xyz="0 0 -0.05" rpy="0 0 0" />
+			<geometry>
+				<box size="10 10 0.1" />
+			</geometry>
+			<material name="IPA/LightGrey"/>
 		</visual>
 	</link>
 	<link name="base_link">
 		<visual>
-		 <origin xyz="0 0 0" rpy="0 0 0" />
-		 <geometry>
-		   <box size="1 0.5 0.5" />
-		 </geometry>
-		 <material name="Red"/>
+			<origin xyz="0 0 0" rpy="0 0 0" />
+			<geometry>
+				<mesh filename="package://cob_description/meshes/base/base.stl"/>
+				<!--box size="1 0.5 0.5" /-->
+			</geometry>
+			<material name="IPA/DarkGrey"/>
 		</visual>
 	</link>
 	<joint name="base_joint" type="floating">
-		<origin xyz="0 0 0.5" rpy="0 0 3.1416"/>
+		<origin xyz="0 0 0" rpy="0 0 0"/>
 		<parent link="map"/>
 		<child link="base_link"/>
